Commit message: Staubli working

File: multiplerobots/urdfFiles/staublirx160/urdf/rx160.urdf (robot description, URDF)
Before this commit: robot staubli_rx160, 8 links, 7 joints
Links:
- added link world
Joints:
- added joint world_base: type fixed, parent world, child base_link, origin xyz=0 0 0 rpy=0 0 0
